File: etc/board/board.kicad_sch (KiCad schematic)
At the start: 10 parts, among them J1 Conn_01x05, U1 Teensy4.1, U2 BOB-09056, U3 TFT_320x240

Commit message: Update code for board v2
Parts:
- removed J1: Conn_01x05, Connector_PinHeader_2.54mm:PinHeader_1x05_P2.54mm_Vertical, symbol Connector_Generic:Conn_01x05
- removed U2: BOB-09056, BOB-09056:MODULE_BOB-09056, symbol BOB-09056:BOB-09056
- R1: footprint Resistor_THT:R_Axial_DIN0204_L3.6mm_D1.6mm_P1.90mm_Vertical -> Resistor_THT:R_Axial_DIN0207_L6.3mm_D2.5mm_P2.54mm_Vertical
- RV1, RV2, RV3, RV4, RV5: footprint Potentiometer_THT:Potentiometer_Omeg_PC16BU_Vertical -> Connector_Molex:Molex_KK-254_AE-6410-03A_1x03_P2.54mm_Vertical
- U3: footprint TFT:TFT-320x240 -> Connector_Molex:Molex_KK-254_AE-6410-14A_1x14_P2.54mm_Vertical
Connections:
- net 3V3: now also U1.15 (3V3)
- net MISO: now reaches U1.14 (12_MISO_MQSL), U3.13
- net MISO: now also U3.9 (MISO)
- net POT3: now reaches RV3.2
- net POT3: now also U1.38 (16_A2_RX4_SCL1)
- net POT2: now reaches RV2.2
- net POT2: now also U1.37 (15_A1_RX3_SPDIF_IN)
- net POT1: now reaches U1.36 (14_A0_TX3_SPDIF_OUT)
- net POT1: now also RV1.2
- net POT4: now reaches U1.39 (17_A3_TX4_SDA1)
- net POT4: now also RV4.2
- net POT5: now reaches U1.44 (22_A8_CTX1)
- net POT5: now also RV5.2
- no-connect marks 0 -> 50
